Commit message: change parameters

File: lite3_urdf/Lite3/urdf/Lite3.urdf (robot description, URDF)
Before this commit: robot MiniLiteV3, 18 links, 17 joints
Joints:
- joint FL_HipX: limit lower=-0.523 upper=0.523 effort=40 velocity=30 -> lower=-0.42 upper=0.42 effort=24 velocity=26
- joint FL_HipY: limit lower=-2.67 upper=0.314 effort=40 velocity=30 -> lower=-2.67 upper=0.314 effort=24 velocity=26
- joint FL_Knee: limit lower=0.524 upper=2.792 effort=65 velocity=20 -> lower=0.6 upper=2.72 effort=36 velocity=17
- joint FR_HipX: limit lower=-0.523 upper=0.523 effort=40 velocity=30 -> lower=-0.42 upper=0.42 effort=24 velocity=26
- joint FR_HipY: limit lower=-2.67 upper=0.314 effort=40 velocity=30 -> lower=-2.67 upper=0.314 effort=24 velocity=26
- joint FR_Knee: limit lower=0.524 upper=2.792 effort=65 velocity=20 -> lower=0.6 upper=2.72 effort=36 velocity=17
- joint HL_HipX: limit lower=-0.523 upper=0.523 effort=40 velocity=30 -> lower=-0.42 upper=0.42 effort=24 velocity=26
- joint HL_HipY: limit lower=-2.67 upper=0.314 effort=40 velocity=30 -> lower=-2.67 upper=0.314 effort=24 velocity=26
- joint HL_Knee: limit lower=0.524 upper=2.792 effort=65 velocity=20 -> lower=0.6 upper=2.72 effort=36 velocity=17
- joint HR_HipX: limit lower=-0.523 upper=0.523 effort=40 velocity=30 -> lower=-0.42 upper=0.42 effort=24 velocity=26
- joint HR_HipY: limit lower=-2.67 upper=0.314 effort=40 velocity=30 -> lower=-2.67 upper=0.314 effort=24 velocity=26
- joint HR_Knee: limit lower=0.524 upper=2.792 effort=65 velocity=20 -> lower=0.6 upper=2.72 effort=36 velocity=17
