Commit message: update x30

File: X30/X30_urdf/urdf/X30.urdf (robot description, URDF)
Before this commit: robot X30, 17 links, 16 joints
Links:
- link FL_SHANK: geometry collision cylinder length=0.08 radius=0.015; collision cylinder length=0.1 radius=0.015
- link FR_SHANK: geometry collision cylinder length=0.08 radius=0.015; collision cylinder length=0.1 radius=0.015
- link HL_SHANK: geometry collision cylinder length=0.08 radius=0.015; collision cylinder length=0.1 radius=0.015
- link HR_SHANK: geometry collision cylinder length=0.08 radius=0.015; collision cylinder length=0.1 radius=0.015

File: X30/X30_urdf/urdf/X30_high_res.urdf (robot description, URDF)
Before this commit: robot X30, 17 links, 16 joints
Links:
- link FL_SHANK: geometry collision cylinder length=0.08 radius=0.015; collision cylinder length=0.1 radius=0.015
- link FR_SHANK: geometry collision cylinder length=0.08 radius=0.015; collision cylinder length=0.1 radius=0.015
- link HL_SHANK: geometry collision cylinder length=0.08 radius=0.015; collision cylinder length=0.1 radius=0.015
- link HR_SHANK: geometry collision cylinder length=0.08 radius=0.015; collision cylinder length=0.1 radius=0.015
