Commit message: Update Lite3 models to the 2026-08-21 OEM release

File: Lite3/urdf/Lite3.urdf (robot description, URDF)
Before this commit: robot Lite3, 17 links, 16 joints
Links:
- added link D435I_LINK
- added link IMU_LINK
- added link MID360_LINK
Joints:
- added joint D435I_FIXED: type fixed, parent TORSO, child D435I_LINK, origin xyz=0.25228 -0.00050 0.07410 rpy=0 -0.3490658504 0
- added joint IMU_FIXED: type fixed, parent TORSO, child IMU_LINK, origin xyz=0.005 0 0 rpy=0 0 0
- added joint MID360_FIXED: type fixed, parent TORSO, child MID360_LINK, origin xyz=0.18678 0 0.12498 rpy=0 -0.2617993878 0

Commit message: Correct Lite3 sensor mount and optical frame orientations
Signed-off-by: Percy <pengbo@deeprobotics.cn>

File: Lite3/urdf/Lite3.urdf (robot description, URDF)
Before this commit: robot Lite3, 20 links, 19 joints
Joints:
- joint D435I_FIXED: origin xyz=0.25228 -0.00050 0.07410 rpy=0 -0.3490658504 0 -> xyz=0.25228 -0.00050 0.07410 rpy=0 0.3490658504 0
- joint MID360_FIXED: origin xyz=0.18678 0 0.12498 rpy=0 -0.2617993878 0 -> xyz=0.18678 0 0.12498 rpy=0 0.2617993878 0
